Commit message: feat: urdf 를 에스뽀 로봇규격에 맞게 설정함.
[설정한 부분]
    - 바퀴와 몸체와 라이다간의 위치 관계

[설정 안한 부분]
    - 캐스터 휠의 위치

File: description/lidar.xacro (robot description, xacro)
@@ -4,5 +4,5 @@
         <parent link="chassis"/>
         <child link="laser_frame"/>
-        <origin xyz="0.122 0 0.212" rpy="0 0 0"/>
+        <origin xyz="0.200 0 0.260" rpy="0 0 0"/>
     </joint>
     <link name="laser_frame">

File: description/robot_core.xacro (robot description, xacro)
@@ -8,9 +8,8 @@
     <xacro:property name="wheel_radius" value="0.0695"/>
     <xacro:property name="wheel_thickness" value="0.063"/>
-    <xacro:property name="wheel_mass" value="2"/>
-    <!-- kg? -->
-    <xacro:property name="wheel_offset_x" value="0.226"/>
+    <xacro:property name="wheel_mass" value="2"/> <!-- kg..? -->
+    <xacro:property name="wheel_offset_x" value="0.1245"/>
     <xacro:property name="wheel_offset_y" value="0.134"/>
-    <xacro:property name="wheel_offset_z" value="0.01"/>
+    <xacro:property name="wheel_offset_z" value="0.02"/>
     <xacro:property name="caster_wheel_radius" value="0.01"/>
     <xacro:property name="caster_wheel_mass" value="0.01"/>
@@ -47,5 +46,5 @@
         <parent link="base_link"/>
         <child link="chassis"/>
-        <origin xyz="${-wheel_offset_x} 0 ${-wheel_offset_z}"/>
+        <origin xyz="${-wheel_offset_x} 0 ${wheel_offset_z}"/>
     </joint>
     <link name="chassis">
